File: DAQSchem/DAQSchem.kicad_sch (KiCad schematic)
At the start: 0 parts

Commit message: Added MCP9600 schematic and I2C pin config
Parts:
- added SCLPull-Up, SDAPull-Up: 4.7K, symbol Device:R
- added U1: STM32F303VCTx, Package_QFP:LQFP-100_14x14mm_P0.5mm, symbol MCU_ST_STM32F3:STM32F303VCTx
- added U2: MCP9600-E_MX, MCP9600-E_MX:QFN65P500X500X100-21N_MCP9600-E_MX, symbol MCP9600-E_MX:MCP9600-E_MX
Connections:
- new net: SCLPull-Up.1, U1.95 (PB8)
- new net: SCLPull-Up.2, U2.19 (SCL)
- new net: U1.49 (VSS), U1.74 (VSS), U1.99 (VSS)
- new net: SDAPull-Up.2, U1.96 (PB9)
- new net: U2.1 (GND), U2.10 (GND), U2.13 (GND), U2.17 (GND), U2.18 (GND), U2.3 (GND), U2.5 (GND), U2.6 (GND), U2.7 (GND), U2.9 (GND)
- new net: SDAPull-Up.1, U2.20 (SDA)
- new net: U2.21 (EXP), U2.22 (EXP), U2.23 (EXP), U2.24 (EXP), U2.25 (EXP), U2.26 (EXP), U2.27 (EXP), U2.28 (EXP), U2.29 (EXP), U2.30 (EXP)
